Commit message: removed redundant meshes folders, changed package name from gp7_description to gp7_visualization

File: gp7_visualization/urdf/gp7_robot.urdf (robot description, URDF)
Before this commit: robot gp7_robot, 7 links, 6 joints
Links:
- link base_link: geometry collision mesh filename=package://gp7_visualization/meshes/collision/base_link.stl; visual mesh filename=package://gp7_visualization/meshes/visual/base_link.STL
- link link_b_5: geometry collision mesh filename=package://gp7_visualization/meshes/collision/link_b_5.stl; visual mesh filename=package://gp7_visualization/meshes/visual/link_b_5.STL
- link link_l_2: geometry collision mesh filename=package://gp7_visualization/meshes/collision/link_l_2.stl; visual mesh filename=package://gp7_visualization/meshes/visual/link_l_2.STL
- link link_r_4: geometry collision mesh filename=package://gp7_visualization/meshes/collision/link_r_4.stl; visual mesh filename=package://gp7_visualization/meshes/visual/link_r_4.STL
- link link_s_1: geometry collision mesh filename=package://gp7_visualization/meshes/collision/link_s_1.stl; visual mesh filename=package://gp7_visualization/meshes/visual/link_s_1.STL
- link link_t_6: geometry collision mesh filename=package://gp7_visualization/meshes/collision/link_t_6.stl; visual mesh filename=package://gp7_visualization/meshes/visual/link_t_6.STL
- link link_u_3: geometry collision mesh filename=package://gp7_visualization/meshes/collision/link_u_3.stl; visual mesh filename=package://gp7_visualization/meshes/visual/link_u_3.STL
