Commit message: fixed link joint names

File: gp7_visualization/urdf/gp7_robot_simple.urdf (robot description, URDF)
Before this commit: robot gp7_robot, 8 links, 7 joints
Links:
- removed link link_1_s
- removed link link_2_l
- removed link link_3_u
- removed link link_4_r
- removed link link_5_b
- removed link link_6_t
- added link link_b_5, mass 0.160644623215161; collision mesh filename=package://gp7_visualization/meshes/collision/link_b_5.stl; visual mesh filename=package://gp7_visualization/meshes/visual/link_b_5.STL
- added link link_l_2, mass 0.562008352548831; collision mesh filename=package://gp7_visualization/meshes/collision/link_l_2.stl; visual mesh filename=package://gp7_visualization/meshes/visual/link_l_2.STL
- added link link_r_4, mass 0.475362712918695; collision mesh filename=package://gp7_visualization/meshes/collision/link_r_4.stl; visual mesh filename=package://gp7_visualization/meshes/visual/link_r_4.STL
- added link link_s_1, mass 0.206747811978373; collision mesh filename=package://gp7_visualization/meshes/collision/link_s_1.stl; visual mesh filename=package://gp7_visualization/meshes/visual/link_s_1.STL
- added link link_t_6, mass 0.0171282195454734; collision mesh filename=package://gp7_visualization/meshes/collision/link_t_6.stl; visual mesh filename=package://gp7_visualization/meshes/visual/link_t_6.STL
- added link link_u_3, mass 0.916688715390813; collision mesh filename=package://gp7_visualization/meshes/collision/link_u_3.stl; visual mesh filename=package://gp7_visualization/meshes/visual/link_u_3.STL
Joints:
- removed joint joint_1_s
- removed joint joint_2_l
- removed joint joint_3_u
- removed joint joint_4_r
- removed joint joint_5_b
- removed joint joint_6_t
- added joint joint_b_5: type revolute, parent link_r_4, child link_b_5, origin xyz=0.11935 0 0 rpy=0 0 0, axis -1 0 0, limit lower=-2.3562 upper=2.3562 effort=17 velocity=9.5993
- added joint joint_l_2: type revolute, parent link_s_1, child link_l_2, origin xyz=0 0 0 rpy=0 0 0, axis 0 -1 0, limit lower=-1.1345 upper=2.5307 effort=30 velocity=6.545
- added joint joint_r_4: type revolute, parent link_u_3, child link_r_4, origin xyz=0.32065 0 0.04 rpy=0 0 0, axis -1 0 0, limit lower=-3.3161 upper=3.3161 effort=17 velocity=9.5993
- added joint joint_s_1: type revolute, parent base_link, child link_s_1, origin xyz=0.039986 -0.0010471 0.33 rpy=0 0 -0.02618, axis 0 0 -1, limit lower=-2.9671 upper=2.9671 effort=30 velocity=6.545
- added joint joint_t_6: type revolute, parent link_b_5, child link_t_6, origin xyz=0.065 0 0 rpy=0 0 0, axis -1 0 0, limit lower=-6.1087 upper=6.1087 effort=10 velocity=17.453
- added joint joint_u_3: type revolute, parent link_l_2, child link_u_3, origin xyz=0 0 0.445 rpy=0 0 0, axis 0 -1 0, limit lower=-1.2217 upper=3.3161 effort=30 velocity=6.545
